Commit message: viualizing camera and laser topic in ROS

File: rrbot_description/model/rrbot.gazebo.xacro (robot description, xacro)
@@ -36,7 +36,7 @@
     <!-- hokuyo -->
     <gazebo reference="${name}_hokuyo_link">
-      <sensor type="gpu_ray" name="head_hokuyo_sensor">
+      <sensor type="ray" name="head_hokuyo_sensor">
         <pose>0 0 0 0 0 0</pose>
-        <visualize>false</visualize>
+        <visualize>true</visualize>
         <update_rate>40</update_rate>
         <ray>
@@ -51,5 +51,5 @@
           <range>
             <min>0.10</min>
-            <max>30.0</max>
+            <max>3.0</max>
             <resolution>0.01</resolution>
           </range>
@@ -64,5 +64,5 @@
           </noise>
         </ray>
-        <plugin name="${name}_gazebo_ros_head_hokuyo_controller" filename="libgazebo_ros_gpu_laser.so">
+        <plugin name="${name}_gazebo_ros_head_hokuyo_controller" filename="libgazebo_ros_laser.so">
           <!-- Publish within the robot namespace -->
           <robotNamespace>${name}</robotNamespace>

File: rrbot_description/model/rrbot.urdf.xacro (robot description, xacro)
@@ -127,5 +127,6 @@
       <origin xyz="0 0 0" rpy="0 0 0"/>
       <geometry>
-        <mesh filename="package://rrbot_description/model/meshes/hokuyo.dae"/>
+        <box size="0.01 0.01 0.01"/>
+        <!--mesh filename="package://rrbot_description/model/meshes/hokuyo.dae"/-->
       </geometry>
     </visual>
@@ -147,5 +148,5 @@
       <origin xyz="0 0 0" rpy="0 0 0"/>
       <geometry>
-	<box size="${camera_link} ${camera_link} ${camera_link}"/>
+        <box size="${camera_link} ${camera_link} ${camera_link}"/>
       </geometry>
     </collision>

File: rrbot_description/robots/single_rrbot.urdf (robot description, URDF)
Before this commit: robot single_rrbot, 6 links, 5 joints
Links:
- link single_rrbot_hokuyo_link: geometry collision box size=0.1 0.1 0.1; visual box size=0.01 0.01 0.01
